Commit message: changes in robot model joints

File: ros2_ws/src/kai/src/description/kai_description.urdf (robot description, URDF)
Before this commit: robot kai, 4 links, 3 joints
Links:
- removed link arm
- removed link servo_motor_1
- removed link servo_motor_2
- added link hand; visual box size=0.05 0.05 0.1
- added link link1; visual box size=0.05 0.05 0.2
- added link link2; visual box size=0.05 0.05 0.2
- added link link3; visual box size=0.05 0.05 0.2
- link base_link: geometry visual box size=0.2 0.2 0.1
Joints:
- removed joint base_to_servo1
- removed joint servo1_to_servo2
- removed joint servo2_to_arm
- added joint joint1: type revolute, parent link1, child link2, origin xyz=0 0 0.2 rpy=0 0 0, axis 0 1 0, limit lower=-1.57 upper=1.57 effort=10 velocity=1
- added joint joint2: type revolute, parent link2, child link3, origin xyz=0 0 0.2 rpy=0 0 0, axis 0 1 0, limit lower=-1.57 upper=1.57 effort=10 velocity=1
- added joint joint3: type revolute, parent link3, child hand, origin xyz=0 0 0.2 rpy=0 0 0, axis 0 1 0, limit lower=-1.57 upper=1.57 effort=10 velocity=1
- added joint primary_joint: type fixed, parent base_link, child link1, origin xyz=0 0 0.1 rpy=0 0 0, axis 0 0 1

Commit message: added robo no working

File: ros2_ws/src/kai/src/description/kai_description.urdf (robot description, URDF)
Before this commit: robot kai, 4 links, 3 joints
Links:
- removed link arm
- removed link servo_motor_1
- removed link servo_motor_2
- added link pen_link; visual cylinder length=0.15 radius=0.01
- added link ruler_link; visual box size=0.3 0.02 0.02
- added link servo_link1; visual box size=0.03 0.03 0.05
- added link servo_link2; visual box size=0.03 0.03 0.05
- link base_link: geometry visual box size=0.1 0.1 0.02
Joints:
- removed joint base_to_servo1
- removed joint servo1_to_servo2
- removed joint servo2_to_arm
- added joint joint1: type continuous, parent base_link, child servo_link1, origin xyz=0 0 0.02 rpy=0 0 0, axis 0 0 1
- added joint joint2: type continuous, parent servo_link1, child servo_link2, origin xyz=0 0 0.05 rpy=0 0 0, axis 0 1 0
- added joint joint3: type fixed, parent servo_link2, child ruler_link, origin xyz=0 0 0.05 rpy=0 0 0
- added joint joint4: type fixed, parent ruler_link, child pen_link, origin xyz=0.15 0 0 rpy=0 0 0
