Commit message: working multi leg robot

File: ros2_ws/src/kai/src/description/robot.urdf (robot description, URDF)
Before this commit: robot onshape, 1 links, 0 joints
Links:
- removed link base
- added link lowerlimb, mass 82.278311597516690767; collision mesh filename=file://$(find kai)/src/description/lowerlimb.stl; visual mesh filename=file://$(find kai)/src/description/lowerlimb.stl
- added link lowerlimb_2, mass 82.278311597516690767; collision mesh filename=file://$(find kai)/src/description/lowerlimb.stl; visual mesh filename=file://$(find kai)/src/description/lowerlimb.stl
- added link lowerlimb_3, mass 82.278311597516690767; collision mesh filename=file://$(find kai)/src/description/lowerlimb.stl; visual mesh filename=file://$(find kai)/src/description/lowerlimb.stl
- added link lowerlimb_4, mass 82.278311597516690767; collision mesh filename=file://$(find kai)/src/description/lowerlimb.stl; visual mesh filename=file://$(find kai)/src/description/lowerlimb.stl
- added link shoulder, mass 10.885618544688634657; collision mesh filename=file://$(find kai)/src/description/shoulder.stl; visual mesh filename=file://$(find kai)/src/description/shoulder.stl
- added link shoulder_2, mass 10.885618544688634657; collision mesh filename=file://$(find kai)/src/description/shoulder.stl; visual mesh filename=file://$(find kai)/src/description/shoulder.stl
- added link shoulder_3, mass 10.885618544688634657; collision mesh filename=file://$(find kai)/src/description/shoulder.stl; visual mesh filename=file://$(find kai)/src/description/shoulder.stl
- added link shoulder_4, mass 10.885618544688634657; collision mesh filename=file://$(find kai)/src/description/shoulder.stl; visual mesh filename=file://$(find kai)/src/description/shoulder.stl
- added link torso_quadruped, mass 229.02210444669583467; collision mesh filename=file://$(find kai)/src/description/torso_quadruped.stl; visual mesh filename=file://$(find kai)/src/description/torso_quadruped.stl
- added link upperlimb, mass 48.066367599923843557; collision mesh filename=file://$(find kai)/src/description/upperlimb.stl; visual mesh filename=file://$(find kai)/src/description/upperlimb.stl
- added link upperlimb_2, mass 48.066367599923843557; collision mesh filename=file://$(find kai)/src/description/upperlimb.stl; visual mesh filename=file://$(find kai)/src/description/upperlimb.stl
- added link upperlimb_3, mass 48.066367599923843557; collision mesh filename=file://$(find kai)/src/description/upperlimb.stl; visual mesh filename=file://$(find kai)/src/description/upperlimb.stl
- added link upperlimb_4, mass 48.066367599923843557; collision mesh filename=file://$(find kai)/src/description/upperlimb.stl; visual mesh filename=file://$(find kai)/src/description/upperlimb.stl
Joints:
- added joint lowerlimb1: type revolute, parent upperlimb, child lowerlimb, origin xyz=8.3266726846886740532e-17 -1.0000000000000004441 3.4694469519536141888e-18 rpy=-3.141592653589793116 7.9073280062811715521e-17 -2.4434609527920607697, axis 0 0 1, limit lower=-2.0943951023931952626 upper=-0.69813170079773179122 effort=1 velocity=20
- added joint lowerlimb2: type revolute, parent upperlimb_2, child lowerlimb_2, origin xyz=5.5511151231257827021e-17 -1 -6.9388939039072283776e-18 rpy=-3.141592653589793116 7.9073280062811740173e-17 -2.4434609527920607697, axis 0 0 1, limit lower=-2.0943951023931952626 upper=-0.69813170079773179122 effort=1 velocity=20
- added joint lowerlimb3: type revolute, parent upperlimb_3, child lowerlimb_3, origin xyz=2.7755575615628913511e-17 1.000000000000000222 -6.9388939039072283776e-18 rpy=3.141592653589793116 4.3391399851923562056e-17 0.69813170079773245735, axis 0 0 1, limit lower=-2.0943951023931952626 upper=-0.69813170079773179122 effort=1 velocity=20
- added joint lowerlimb4: type revolute, parent upperlimb_4, child lowerlimb_4, origin xyz=2.7755575615628913511e-16 0.99999999999999988898 3.4694469519536141888e-18 rpy=3.141592653589793116 4.339139985192361136e-17 0.69813170079773234633, axis 0 0 1, limit lower=-2.0943951023931952626 upper=-0.69813170079773179122 effort=1 velocity=20
- added joint shoulder1: type revolute, parent torso_quadruped, child shoulder, origin xyz=0.3638696238398552163 0.030409909784793860699 0.15190468430519105114 rpy=3.141592653589793116 -0 0, axis 0 0 1, limit lower=-0.785398163397448279 upper=0.785398163397448279 effort=1 velocity=20
- added joint shoulder2: type revolute, parent torso_quadruped, child shoulder_2, origin xyz=-0.036130376160144812847 0.43040990978479387596 0.15190468430519105114 rpy=3.141592653589793116 -0 1.570796326794896558, axis 0 0 1, limit lower=-0.785398163397448279 upper=0.785398163397448279 effort=1 velocity=20
- added joint shoulder3: type revolute, parent torso_quadruped, child shoulder_3, origin xyz=-0.036130376160144798969 -0.36959009021520616844 0.15190468430519105114 rpy=3.141592653589793116 -0 -1.570796326794896558, axis 0 0 1, limit lower=-0.785398163397448279 upper=0.785398163397448279 effort=1 velocity=20
- added joint shoulder4: type revolute, parent torso_quadruped, child shoulder_4, origin xyz=-0.43613037616014482811 0.030409909784793846821 0.15190468430519105114 rpy=3.141592653589793116 -0 3.141592653589793116, axis 0 0 1, limit lower=-0.785398163397448279 upper=0.785398163397448279 effort=1 velocity=20
- added joint upperlimb1: type revolute, parent shoulder, child upperlimb, origin xyz=0 6.9388939039072283776e-18 -0.1500000000000000222 rpy=1.570796326794896558 0.34906585039886578459 3.141592653589793116, axis 0 0 1, limit lower=-1.570796326794896558 upper=-0.34906585039886589561 effort=1 velocity=20
- added joint upperlimb2: type revolute, parent shoulder_2, child upperlimb_2, origin xyz=0 6.9388939039072283776e-18 -0.1500000000000000222 rpy=1.570796326794896558 0.34906585039886578459 3.141592653589793116, axis 0 0 1, limit lower=-1.570796326794896558 upper=-0.34906585039886589561 effort=1 velocity=20
- added joint upperlimb3: type revolute, parent shoulder_3, child upperlimb_3, origin xyz=-5.5511151231257827021e-17 6.9388939039072283776e-18 -0.15000000000000007772 rpy=-1.570796326794896558 -0.34906585039886578459 6.5162095139319294904e-17, axis 0 0 1, limit lower=-1.570796326794896558 upper=-0.34906585039886589561 effort=1 velocity=20
- added joint upperlimb4: type revolute, parent shoulder_4, child upperlimb_4, origin xyz=-5.5511151231257827021e-17 6.9388939039072283776e-18 -0.14999999999999985567 rpy=-1.570796326794896558 -0.34906585039886578459 6.5162095139319294904e-17, axis 0 0 1, limit lower=-1.570796326794896558 upper=-0.34906585039886589561 effort=1 velocity=20

Commit message: added gazebo

File: ros2_ws/src/kai/src/description/robot.urdf (robot description, URDF)
Before this commit: robot onshape, 5 links, 4 joints
Joints:
- removed joint outarm
- added joint outarm_joint: type revolute, parent assembly_1, child outarm, origin xyz=-3.9621084191310274036e-15 0.099034298211335899942 0.044499999999999789724 rpy=-3.1415926535897900074 -2.1456705084130752623e-15 0.77445109514413923435, axis 0 0 1, limit lower=-1.0 upper=2.141592653589793116 effort=1 velocity=20

Commit message: hi

File: ros2_ws/src/kai/src/description/robot.urdf (robot description, URDF)
Before this commit: robot kai, 5 links, 4 joints
Links:
- removed link assembly_1
- removed link assembly_2
- removed link mg995
- added link Base, mass 0.38937999999999994838; collision mesh filename=file://$(find kai)/src/description/base.stl; collision mesh filename=file://$(find kai)/src/description/mg995.stl
- added link Hand, mass 0.070766740240779890669; collision mesh filename=file://$(find kai)/src/description/mg995.stl; collision mesh filename=file://$(find kai)/src/description/outarm.stl
- added link Servo, mass 0.058000000000000002942; collision mesh filename=file://$(find kai)/src/description/mg995.stl; visual mesh filename=file://$(find kai)/src/description/mg995.stl
- added link dummy_link, mass 0.1
- link baselink: mass 1e-9 -> 0.1
Joints:
- removed joint baselink_frame
- removed joint baseyaw
- removed joint motor2
- added joint Base_joint: type fixed, parent Base, child baselink, origin xyz=-0.010000000000000000208 -1.3877787807814442889e-17 -0.072000000000000036193 rpy=-2.3111159332646792604e-33 -1.2325951644078287564e-32 -1.570796326794896558, axis 0 0 0
- added joint Hand_joint: type revolute, parent Servo, child Hand, origin xyz=-0.01941721109241918708 -0.012625212490669088933 0.079500000000000237144 rpy=1.5707963267948970021 -0.45450288711037684086 2.0903181118752649503, axis 0 0 1, limit lower=-2.0 upper=1.141592653589793116 effort=1 velocity=20
- added joint Motor_joint: type revolute, parent Servo, child Base, origin xyz=-1.3877787807814456755e-17 0.010000000000000005412 0.06950000000000011724 rpy=1.2325951644078287564e-32 -2.3111159332646792604e-33 1.570796326794896558, axis 0 0 1, limit lower=0 upper=3.141592653589793116 effort=1 velocity=20
- added joint dummy_joint: type fixed, parent dummy_link, child Servo, origin xyz=0 0 0 rpy=0 0 0
- joint outarm_joint: parent assembly_1 -> Hand
