Commit message: controllers working

File: ros2_ws/src/kai/src/description/gazebo.xacro (robot description, xacro)
@@ -1,4 +1,9 @@
 <?xml version="1.0" ?>
 <robot xmlns:xacro="http://www.ros.org/wiki/xacro">
+<gazebo>
+        <plugin filename="ign_ros2_control-system" name="ign_ros2_control::IgnitionROS2ControlPlugin">
+            <parameters>$(find kai)/config/kai_controller.yaml</parameters>
+        </plugin>
+    </gazebo>
 <gazebo reference="outarm">
   <material>Gazebo/Red</material>

File: ros2_ws/src/kai/src/description/robot.urdf.xacro (robot description, xacro)
@@ -1,6 +1,6 @@
 <?xml version="1.0"?>
 <robot xmlns:xacro="http://www.ros.org/wiki/xacro"  name="kai">
-<xacro:include filename="robot_core.xacro" />
-<xacro:include filename="gazebo.xacro" />
-<xacro:include filename="ros_control.xacro" />
+<xacro:include filename="$(find kai)/src/description/robot_core.xacro" />
+<xacro:include filename="$(find kai)/src/description/gazebo.xacro" />
+<xacro:include filename="$(find kai)/src/description/ros_control.xacro" />
 </robot>

File: ros2_ws/src/kai/src/description/robot_core.xacro (robot description, xacro)
@@ -119,7 +119,7 @@
 </inertial>
 </link>
-<link name="baselink" />
+<link name="world" />
 <joint name="baselink_frame" type="fixed">
-<parent link="baselink" />
+<parent link="world" />
 <child link="base" />
 <axis xyz="0 0 0"/>
@@ -131,5 +131,5 @@
 <axis xyz="0 0 1"/>
 <limit effort="1" velocity="20" lower="0" upper="3.141592653589793116"/>
-<joint_properties friction="0.0"/>
+<dynamics damping="0.05" friction="0.05"/>
 </joint>
 <joint name="outarm_joint" type="revolute">
@@ -139,5 +139,5 @@
 <axis xyz="0 0 1"/>
 <limit effort="1" velocity="20" lower="-1.0" upper="2.141592653589793116"/>
-<joint_properties friction="0.0"/>
+<dynamics damping="0.05" friction="0.05"/>
 </joint>
 <joint name="baseroll_joint" type="revolute">
@@ -147,5 +147,5 @@
 <axis xyz="0 0 1"/>
 <limit effort="1" velocity="20" lower="-2.0" upper="1.141592653589793116"/>
-<joint_properties friction="0.0"/>
+<dynamics damping="0.05" friction="0.05"/>
 </joint>
 <!-- <gazebo>

File: ros2_ws/src/kai/src/description/ros_control.xacro (robot description, xacro)
@@ -3,9 +3,9 @@
 <ros2_control name="kai_controller" type="system">
  <hardware>
-   <plugin>mock_components/GenericSystem</plugin>
+   <plugin>ign_ros2_control/IgnitionSystem</plugin>
    <param name="example_param_write_for_sec">2</param>
    <param name="example_param_read_for_sec">2</param>
  </hardware>
- <joint name="baseyaw">
+ <joint name="baseyaw_joint">
    <command_interface name="position">
      <param name="min">0</param>
@@ -14,5 +14,5 @@
    <state_interface name="position"/>
  </joint>
- <joint name="motor2">
+ <joint name="baseroll_joint">
    <command_interface name="position">
      <param name="min">-2</param>

Commit message: fixed gazebo

File: ros2_ws/src/kai/src/description/gazebo.xacro (robot description, xacro)
@@ -8,6 +8,6 @@
 <gazebo reference="outarm">
   <material>Gazebo/Red</material>
-  <mu1>0.2</mu1>
-  <mu2>0.2</mu2>
+  <!-- <mu1>0.2</mu1>
+  <mu2>0.2</mu2> -->
   <self_collide>true</self_collide>
   <gravity>true</gravity>
@@ -15,6 +15,6 @@
 <gazebo reference="base">
   <material>Gazebo/Black</material>
-  <mu1>0.2</mu1>
-  <mu2>0.2</mu2>
+  <!-- <mu1>0.2</mu1>
+  <mu2>0.2</mu2> -->
   <self_collide>true</self_collide>
   <gravity>true</gravity>
@@ -22,6 +22,6 @@
 <gazebo reference="upperarm">
   <material>Gazebo/Black</material>
-  <mu1>0.2</mu1>
-  <mu2>0.2</mu2>
+  <!-- <mu1>0.2</mu1>
+  <mu2>0.2</mu2> -->
   <self_collide>true</self_collide>
   <gravity>true</gravity>
@@ -29,6 +29,6 @@
 <gazebo reference="mg995">
   <material>Gazebo/Black</material>
-  <mu1>0.2</mu1>
-  <mu2>0.2</mu2>
+  <!-- <mu1>0.2</mu1>
+  <mu2>0.2</mu2> -->
   <self_collide>true</self_collide>
   <gravity>true</gravity>

File: ros2_ws/src/kai/src/description/robot_core.xacro (robot description, xacro)
@@ -130,5 +130,5 @@
 <child link="mg995" />
 <axis xyz="0 0 1"/>
-<limit effort="1" velocity="20" lower="0" upper="3.14"/>
+<limit effort="1" velocity="20" lower="0" upper="3.141592653589793116"/>
 <dynamics damping="0.05" friction="0.05"/>
 </joint>
@@ -149,8 +149,3 @@
 <dynamics damping="0.05" friction="0.05"/>
 </joint>
-<!-- <gazebo>
-    <plugin filename="ign_ros2_control-system" name="ign_ros2_control::IgnitionROS2ControlPlugin">
-     <parameters>$(find kai)/config/kai_controller.yaml</parameters>
-    </plugin>
-</gazebo> -->
 </robot>

File: ros2_ws/src/kai/src/description/ros_control.xacro (robot description, xacro)
@@ -3,5 +3,6 @@
 <ros2_control name="kai_controller" type="system">
  <hardware>
-   <plugin>kai/RobotSystem</plugin>
+   <!-- <plugin>kai/RobotSystem</plugin> -->
+   <plugin>ign_ros2_control/IgnitionSystem</plugin>
    <param name="example_param_write_for_sec">2</param>
    <param name="example_param_read_for_sec">2</param>
