Commit message: working hardware

File: ros2_ws/src/kai/src/description/robot_core.xacro (robot description, xacro)
@@ -130,5 +130,5 @@
 <child link="mg995" />
 <axis xyz="0 0 1"/>
-<limit effort="1" velocity="20" lower="0" upper="3.141592653589793116"/>
+<limit effort="1" velocity="20" lower="0" upper="3.14"/>
 <dynamics damping="0.05" friction="0.05"/>
 </joint>

File: ros2_ws/src/kai/src/description/ros_control.xacro (robot description, xacro)
@@ -3,5 +3,5 @@
 <ros2_control name="kai_controller" type="system">
  <hardware>
-   <plugin>ign_ros2_control/IgnitionSystem</plugin>
+   <plugin>kai/RobotSystem</plugin>
    <param name="example_param_write_for_sec">2</param>
    <param name="example_param_read_for_sec">2</param>

Commit message: moveit hardware plugin

File: ros2_ws/src/kai/src/description/robot_core.xacro (robot description, xacro)
@@ -119,10 +119,5 @@
 </inertial>
 </link>
-<link name="world" />
-<joint name="baselink_frame" type="fixed">
-<parent link="world" />
-<child link="base" />
-<axis xyz="0 0 0"/>
-</joint>
+<link name="endeffector"/>
 <joint name="baseyaw_joint" type="revolute">
 <origin xyz="0 0 0.065" rpy="1.2325951644078287564e-32 -2.3111159332646792604e-33 1.570796326794896558" />
@@ -130,5 +125,5 @@
 <child link="mg995" />
 <axis xyz="0 0 1"/>
-<limit effort="1" velocity="20" lower="0" upper="3.141592653589793116"/>
+<limit effort="1.0" velocity="20.01" lower="0" upper="3.141592653589793116"/>
 <dynamics damping="0.05" friction="0.05"/>
 </joint>
@@ -138,6 +133,11 @@
 <child link="outarm" />
 <axis xyz="0 0 1"/>
-<limit effort="1" velocity="20" lower="-1.0" upper="2.141592653589793116"/>
+<limit effort="1.0" velocity="20.01" lower="-1.0" upper="2.141592653589793116"/>
 <dynamics damping="0.05" friction="0.05"/>
+</joint>
+<joint name="endeffector_joint" type="fixed">
+<origin xyz="0.075 0 0"/>
+<parent link="outarm" />
+<child link="endeffector" />
 </joint>
 <joint name="baseroll_joint" type="revolute">
@@ -146,5 +146,5 @@
 <child link="upperarm" />
 <axis xyz="0 0 1"/>
-<limit effort="1" velocity="20" lower="-2.0" upper="1.141592653589793116"/>
+<limit effort="1.0" velocity="20.01" lower="-2.0" upper="1.141592653589793116"/>
 <dynamics damping="0.05" friction="0.05"/>
 </joint>

File: ros2_ws/src/kai/src/description/ros_control.xacro (robot description, xacro)
@@ -3,6 +3,6 @@
 <ros2_control name="kai_controller" type="system">
  <hardware>
-   <!-- <plugin>kai/RobotSystem</plugin> -->
-   <plugin>ign_ros2_control/IgnitionSystem</plugin>
+   <plugin>kai/RobotSystem</plugin>
+   <!-- <plugin>ign_ros2_control/IgnitionSystem</plugin> -->
    <param name="example_param_write_for_sec">2</param>
    <param name="example_param_read_for_sec">2</param>
