Commit message: fixed description package

File: ros2_ws/r6bot.urdf (robot description, URDF)
Before this commit: robot kai, 5 links, 4 joints
Links:
- removed link assembly_1
- removed link assembly_2
- added link base, mass 0.38937999999999994838; collision mesh filename=file:///home/prasannan-robot/Desktop/Papi/ros2_ws/install/k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; collision mesh filename=file:///home/prasannan-robot/Desktop/Papi/ros2_ws/install/k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
- added link upperarm, mass 0.070766740240779890669; collision mesh filename=file:///home/prasannan-robot/Desktop/Papi/ros2_ws/install/k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; collision mesh filename=file:///home/prasannan-robot/Desktop/Papi/ros2_ws/install/k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
- link baselink: mass 1e-9 -> None
Joints:
- removed joint baseyaw
- removed joint motor2
- added joint baseroll_joint: type revolute, parent mg995, child upperarm, origin xyz=-0.01941721109241918708 -0.012625212490669088933 0.009 rpy=1.5707963267948970021 -0.45450288711037684086 2.0903181118752649503, axis 0 0 1, limit lower=-2.0 upper=1.141592653589793116 effort=1 velocity=20
- added joint baseyaw_joint: type revolute, parent base, child mg995, origin xyz=0 0 0.065 rpy=1.2325951644078287564e-32 -2.3111159332646792604e-33 1.570796326794896558, axis 0 0 1, limit lower=0 upper=3.141592653589793116 effort=1 velocity=20
- joint baselink_frame: child baselink -> base; origin xyz=-0.010000000000000000208 -1.3877787807814442889e-17 -0.072000000000000036193 rpy=-2.3111159332646792604e-33 -1.2325951644078287564e-32 -1.570796326794896558 -> (none); parent assembly_2 -> baselink
- joint outarm_joint: origin xyz=-3.9621084191310274036e-15 0.099034298211335899942 0.044499999999999789724 rpy=-3.1415926535897900074 -2.1456705084130752623e-15 0.77445109514413923435 -> xyz=-3.9621084191310274036e-15 0.099034298211335899942 0.043 rpy=-3.1415926535897900074 -2.1456705084130752623e-15 0.77445109514413923435; parent assembly_1 -> upperarm
