Commit message: [Feat] added gantry

File: ros2_ws/src/hath/src/description/robot.urdf (robot description, URDF)
Before this commit: robot onshape, 4 links, 3 joints
Links:
- link e1: geometry collision mesh filename=file://$(find hath)/src/description/meshes/e1.stl; visual mesh filename=file://$(find hath)/src/description/meshes/e1.stl
- link e2: geometry collision mesh filename=file://$(find hath)/src/description/meshes/e2.stl; visual mesh filename=file://$(find hath)/src/description/meshes/e2.stl
- link e3: geometry collision mesh filename=file://$(find hath)/src/description/meshes/e3.stl; visual mesh filename=file://$(find hath)/src/description/meshes/e3.stl
- link e4: geometry collision mesh filename=file://$(find hath)/src/description/meshes/e4.stl; visual mesh filename=file://$(find hath)/src/description/meshes/e4.stl
Joints:
- joint x: limit lower=0.010000000000000000208 upper=0.83999999999999996891 effort=1 velocity=20 -> lower=0.0 upper=0.630 effort=1 velocity=20; origin xyz=0.14338706748580448691 0.4749999999999999778 0.60499999999999998224 rpy=1.570796326794896558 -0 -1.570796326794896558 -> xyz=0.400 0.4749999999999999778 0.60499999999999998224 rpy=1.570796326794896558 -0 -1.570796326794896558
- joint z: limit lower=0.10000000000000000555 upper=0.69999999999999995559 effort=1 velocity=20 -> lower=-0.100 upper=0.159 effort=1 velocity=20

Commit message: added gazebo

File: ros2_ws/src/hath/src/description/robot.urdf (robot description, URDF)
Before this commit: robot onshape, 4 links, 3 joints
Joints:
- removed joint y
- added joint y_axis: type prismatic, parent e2, child e3, origin xyz=0.86499999999999876987 0 0.025000000000000008327 rpy=-1.570796326794896558 -1.065814103631468549e-14 1.5707963267949136554, axis 0 0 1, limit lower=0.05999999999999999778 upper=0.83999999999999996891 effort=100 velocity=200
- joint x: limit lower=0.0 upper=0.630 effort=1 velocity=20 -> lower=0.0 upper=0.630 effort=100 velocity=200
- joint z: limit lower=-0.100 upper=0.159 effort=1 velocity=20 -> lower=-0.100 upper=0.159 effort=100 velocity=200
