Commit message: little progress

File: arm/robot.urdf (robot description, URDF)
Before this commit: robot onshape, 15 links, 14 joints
Links:
- removed link body
- removed link doubleu
- removed link doubleu_2
- removed link doubleu_3
- removed link doubleu_4
- removed link leg
- removed link leg_2
- removed link leg_3
- removed link leg_4
- removed link platesblock
- removed link platesblock_2
- removed link platesblock_3
- removed link platesblock_4
- removed link tip
- removed link trunk
- added link assembly_1, mass 0.070766740240779890669; collision mesh filename=package:///mg995.stl; collision mesh filename=package:///outarm.stl
- added link base, mass 1e-9
- added link mg995, mass 0.058000000000000002942; collision mesh filename=package:///mg995.stl; visual mesh filename=package:///mg995.stl
- added link mg995_2, mass 0.058000000000000002942; collision mesh filename=package:///mg995.stl; visual mesh filename=package:///mg995.stl
- added link outarm, mass 0.012766740240779891197; collision mesh filename=package:///outarm.stl; visual mesh filename=package:///outarm.stl
Joints:
- removed joint leg1_a
- removed joint leg1_b
- removed joint leg1_c
- removed joint leg2_a
- removed joint leg2_b
- removed joint leg2_c
- removed joint leg3_a
- removed joint leg3_b
- removed joint leg3_c
- removed joint leg4_a
- removed joint leg4_b
- removed joint leg4_c
- removed joint tip_frame
- removed joint trunk_frame
- added joint base_frame: type fixed, parent mg995_2, child base, origin xyz=-0.010000000000000000208 0.0022040872588557753296 -0.069499999999999992339 rpy=5.3926038442842590201e-33 -5.3926038442842289141e-33 -1.570796326794896558, axis 0 0 0
- added joint baseyaw: type revolute, parent mg995, child mg995_2, origin xyz=-1.3877787807814456755e-17 0.010000000000000005412 0.06950000000000011724 rpy=1.2325951644078287564e-32 -2.3111159332646792604e-33 1.570796326794896558, axis 0 0 1, limit lower=0 upper=3.141592653589793116 effort=1 velocity=20
- added joint motor2: type revolute, parent mg995, child assembly_1, origin xyz=-0.01941721109241918708 -0.012625212490669088933 0.079500000000000237144 rpy=1.5707963267948970021 -0.45450288711037684086 2.0903181118752649503, axis 0 0 1, limit lower=0 upper=3.141592653589793116 effort=1 velocity=20
- added joint outarm: type revolute, parent assembly_1, child outarm, origin xyz=-3.9621084191310274036e-15 0.099034298211335899942 0.044499999999999789724 rpy=-3.1415926535897900074 -2.1456705084130752623e-15 0.77445109514413923435, axis 0 0 1, limit lower=0 upper=3.141592653589793116 effort=1 velocity=20

File: ros2_ws/src/kai/src/description/robot.urdf (robot description, URDF)
Before this commit: robot quadruped_robot, 13 links, 12 joints
Links:
- removed link lowerlimb
- removed link lowerlimb_2
- removed link lowerlimb_3
- removed link lowerlimb_4
- removed link shoulder
- removed link shoulder_2
- removed link shoulder_3
- removed link shoulder_4
- removed link torso_quadruped
- removed link upperlimb
- removed link upperlimb_2
- removed link upperlimb_3
- removed link upperlimb_4
- added link assembly_1, mass 0.070766740240779890669; collision mesh filename=file://$(find kai)/src/description/mg995.stl; collision mesh filename=file://$(find kai)/src/description/outarm.stl
- added link mg995, mass 0.058000000000000002942; collision mesh filename=file://$(find kai)/src/description/mg995.stl; visual mesh filename=file://$(find kai)/src/description/mg995.stl
- added link mg995_2, mass 0.38937999999999994838; collision mesh filename=file://$(find kai)/src/description/base.stl; collision mesh filename=file://$(find kai)/src/description/mg995.stl
- added link outarm, mass 0.012766740240779891197; collision mesh filename=file://$(find kai)/src/description/outarm.stl; visual mesh filename=file://$(find kai)/src/description/outarm.stl
Joints:
- removed joint lowerlimb1
- removed joint lowerlimb2
- removed joint lowerlimb3
- removed joint lowerlimb4
- removed joint shoulder1
- removed joint shoulder2
- removed joint shoulder3
- removed joint shoulder4
- removed joint upperlimb1
- removed joint upperlimb2
- removed joint upperlimb3
- removed joint upperlimb4
- added joint base: type revolute, parent mg995, child assembly_1, origin xyz=0.028570946193171013749 0.0015843545963584067249 0.079590287562755684947 rpy=-1.570796326794896558 -0.019341669366944650582 0.94518153198707821616, axis 0 0 1, limit effort=1 velocity=20
- added joint baseyaw: type revolute, parent mg995, child mg995_2, origin xyz=-6.9611571409717492764e-18 0.010000000000000005412 0.069500000000000089484 rpy=1.2325951644078287564e-32 -2.3111159332646792604e-33 1.570796326794896558, axis 0 0 1, limit lower=0 upper=3.141592653589793116 effort=1 velocity=20
- added joint outarm: type revolute, parent assembly_1, child outarm, origin xyz=-3.6706748751669238118e-15 -0.099034298211335927697 -0.049499999999999128031 rpy=-4.1390834984404515333e-15 -1.0914910073606571169e-15 -1.6138091426053176036, axis 0 0 1, limit lower=0 upper=3.141592653589793116 effort=1 velocity=20

Commit message: working urdf but transform issue

File: arm/robot.urdf (robot description, URDF)
Before this commit: robot onshape, 5 links, 4 joints
Links:
- removed link base
- removed link mg995_2
- added link assembly_2, mass 0.38937999999999994838; collision mesh filename=package:///base.stl; collision mesh filename=package:///mg995.stl
- added link baselink, mass 1e-9
- link outarm: mass 0.012766740240779891197 -> 0.012766740240779889462
Joints:
- removed joint base_frame
- added joint baselink_frame: type fixed, parent assembly_2, child baselink, origin xyz=-0.010000000000000000208 -1.3877787807814442889e-17 -0.072000000000000036193 rpy=-2.3111159332646792604e-33 -1.2325951644078287564e-32 -1.570796326794896558, axis 0 0 0
- joint baseyaw: child mg995_2 -> assembly_2

File: ros2_ws/src/kai/src/description/robot.urdf (robot description, URDF)
Before this commit: robot onshape, 4 links, 3 joints
Links:
- link mg995_2: mass 0.38937999999999994838 -> 0.38938000000000000389
- link outarm: mass 0.012766740240779891197 -> 0.012766740240779889462
Joints:
- removed joint base
- added joint motor2: type revolute, parent mg995, child assembly_1, origin xyz=-0.01941721109241918708 -0.012625212490669088933 0.079500000000000237144 rpy=1.5707963267948970021 -0.45450288711037684086 2.0903181118752649503, axis 0 0 1, limit lower=0 upper=3.141592653589793116 effort=1 velocity=20
- joint baseyaw: origin xyz=-6.9611571409717492764e-18 0.010000000000000005412 0.069500000000000089484 rpy=1.2325951644078287564e-32 -2.3111159332646792604e-33 1.570796326794896558 -> xyz=-1.3877787807814456755e-17 0.010000000000000005412 0.06950000000000011724 rpy=1.2325951644078287564e-32 -2.3111159332646792604e-33 1.570796326794896558
- joint outarm: origin xyz=-3.6706748751669238118e-15 -0.099034298211335927697 -0.049499999999999128031 rpy=-4.1390834984404515333e-15 -1.0914910073606571169e-15 -1.6138091426053176036 -> xyz=-3.9621084191310274036e-15 0.099034298211335899942 0.044499999999999789724 rpy=-3.1415926535897900074 -2.1456705084130752623e-15 0.77445109514413923435

Commit message: urdf finished

File: arm/robot.urdf (robot description, URDF)
Before this commit: robot onshape, 5 links, 4 joints
Links:
- link assembly_1: geometry collision mesh filename=file://$(find kai)/src/description/mg995.stl; collision mesh filename=file://$(find kai)/src/description/outarm.stl
- link assembly_2: geometry collision mesh filename=file://$(find kai)/src/description/base.stl; collision mesh filename=file://$(find kai)/src/description/mg995.stl
- link mg995: geometry collision mesh filename=file://$(find kai)/src/description/mg995.stl; visual mesh filename=file://$(find kai)/src/description/mg995.stl
- link outarm: geometry collision mesh filename=file://$(find kai)/src/description/outarm.stl; visual mesh filename=file://$(find kai)/src/description/outarm.stl

File: ros2_ws/src/kai/src/description/robot.urdf (robot description, URDF)
Before this commit: robot onshape, 4 links, 3 joints
Links:
- removed link mg995_2
- added link assembly_2, mass 0.38937999999999994838; collision mesh filename=file://$(find kai)/src/description/base.stl; collision mesh filename=file://$(find kai)/src/description/mg995.stl
- added link baselink, mass 1e-9
Joints:
- added joint baselink_frame: type fixed, parent assembly_2, child baselink, origin xyz=-0.010000000000000000208 -1.3877787807814442889e-17 -0.072000000000000036193 rpy=-2.3111159332646792604e-33 -1.2325951644078287564e-32 -1.570796326794896558, axis 0 0 0
- joint baseyaw: child mg995_2 -> assembly_2
- joint motor2: limit lower=0 upper=3.141592653589793116 effort=1 velocity=20 -> lower=-2.0 upper=1.141592653589793116 effort=1 velocity=20
- joint outarm: limit lower=0 upper=3.141592653589793116 effort=1 velocity=20 -> lower=-1.0 upper=2.141592653589793116 effort=1 velocity=20

Commit message: some changes

File: arm/robot.urdf (robot description, URDF)
Before this commit: robot onshape, 5 links, 4 joints
Links:
- removed link assembly_1
- removed link assembly_2
- removed link baselink
- added link arm, mass 0.070766740240779890669; collision mesh filename=package:///mg995.stl; collision mesh filename=package:///outarm.stl
- added link base_assembly, mass 0.38938000000000000389; collision mesh filename=package:///base.stl; collision mesh filename=package:///mg995.stl
- link mg995: geometry collision mesh filename=package:///mg995.stl; visual mesh filename=package:///mg995.stl
- link outarm: mass 0.012766740240779889462 -> 0.012766740240779891197; geometry collision mesh filename=package:///outarm.stl; visual mesh filename=package:///outarm.stl
Joints:
- removed joint baselink_frame
- removed joint motor2
- removed joint outarm
- added joint armpitch: type revolute, parent arm, child outarm, origin xyz=-4.8468173918791990218e-15 0.099034298211335955453 0.044500000000000275446 rpy=-3.1415926535897926719 -6.9474246886750598283e-18 -3.141592653589793116, axis 0 0 1, limit lower=0 upper=3.141592653589793116 effort=1 velocity=20
- added joint basepitch: type revolute, parent mg995, child arm, origin xyz=-0.020000000000000014294 0.028087867965644174734 0.07950000000000032041 rpy=1.5707963267948923392 1.6653345369377614347e-16 1.4447285194009526164e-15, axis 0 0 1, limit lower=0 upper=3.141592653589793116 effort=1 velocity=20
- joint baseyaw: child assembly_2 -> base_assembly; origin xyz=-1.3877787807814456755e-17 0.010000000000000005412 0.06950000000000011724 rpy=1.2325951644078287564e-32 -2.3111159332646792604e-33 1.570796326794896558 -> xyz=-0.010000000000000045311 1.7249945589578561902e-16 0.06950000000000049194 rpy=-5.5511151231269881802e-17 -4.9404924595819963031e-15 -3.1415926535897917837

Commit message: [Feat Bar] New Cad

File: arm/robot.urdf (robot description, URDF)
Before this commit: robot onshape, 4 links, 3 joints
Links:
- removed link e1
- removed link e2
- removed link e3
- removed link e4
- added link 8mmrod1, mass 8.6576870598331243656; collision mesh filename=package:///8mmrod1.stl; collision mesh filename=package:///8mmrod2.stl
- added link part_3, mass 0.31828084038355258789; collision mesh filename=package:///part_2.stl; collision mesh filename=package:///part_3.stl
Joints:
- removed joint x
- removed joint y
- removed joint z
- added joint sliderx: type prismatic, parent 8mmrod1, child part_3, origin xyz=-0.25000000000000177636 -0.24999999999999991673 0.64499999999999890754 rpy=-1.570796326794911435 1.8608419724351648241e-15 1.570796326794896336, axis 0 0 1, limit lower=-0.19000000000000000222 upper=0.23000000000000000999 effort=1 velocity=20

File: ros2_ws/src/hath/src/description/robot.urdf (robot description, URDF)
Before this commit: robot onshape, 4 links, 3 joints
Links:
- removed link e1
- removed link e2
- removed link e3
- removed link e4
- added link 8mmrod1, mass 8.6576870598331243656; collision mesh filename=file://$(find hath)/src/description/meshes/8mmrod1.stl; collision mesh filename=file://$(find hath)/src/description/meshes/8mmrod2.stl
- added link part_3, mass 0.31828084038355258789; collision mesh filename=file://$(find hath)/src/description/meshes/part_2.stl; collision mesh filename=file://$(find hath)/src/description/meshes/part_3.stl
Joints:
- removed joint x
- removed joint y_axis
- removed joint z
- added joint sliderx: type prismatic, parent 8mmrod1, child part_3, origin xyz=-0.25000000000000177636 -0.24999999999999991673 0.64499999999999890754 rpy=-1.570796326794911435 1.8608419724351648241e-15 1.570796326794896336, axis 0 0 1, limit lower=-0.19000000000000000222 upper=0.23000000000000000999 effort=1 velocity=20

Commit message: enanu therla

File: arm/robot.urdf (robot description, URDF)
Before this commit: robot onshape, 2 links, 1 joints
Links:
- removed link 8mmrod1
- removed link part_3
- added link part_2_lf, mass 0.361099999999999699; collision mesh filename=package:///part_12.stl; collision mesh filename=package:///part_2_lf.stl
- added link part_2_lf_2, mass 0.36109999999999964349; collision mesh filename=package:///part_2_lf.stl; collision mesh filename=package:///part_2_lf.stl
Joints:
- joint sliderx: child part_3 -> part_2_lf_2; limit lower=-0.19000000000000000222 upper=0.23000000000000000999 effort=1 velocity=20 -> lower=-0.022 upper=0.199 effort=1 velocity=20; origin xyz=-0.25000000000000177636 -0.24999999999999991673 0.64499999999999890754 rpy=-1.570796326794911435 1.8608419724351648241e-15 1.570796326794896336 -> xyz=0.0099999999999999811262 -0.13999999999999998557 0.0099999999999999984734 rpy=1.9721522630525295135e-31 1.570796326794896558 0; parent 8mmrod1 -> part_2_lf

File: ros2_ws/src/hath/src/description/robot.urdf (robot description, URDF)
Before this commit: robot onshape, 2 links, 1 joints
Links:
- removed link 8mmrod1
- removed link part_3
- added link bottomplate, mass 39.717716802635088413; collision mesh filename=file://$(find hath)/src/description/meshes/8mmrod.stl; collision mesh filename=file://$(find hath)/src/description/meshes/8mmrod.stl
Joints:
- removed joint sliderx
